Commit message: add rotations, fix round-robin sampling, update gifs

File: source/assets/piper_x/piper_x_d435.urdf (robot description, URDF)
Before this commit: robot piper_x_camera, 13 links, 12 joints
Links:
- link Link8: geometry collision mesh filename=meshes/J7.dae; visual mesh filename=meshes/J8.dae
